File: hb_chip_test/hb_chip_test.kicad_pcb (KiCad board)
At the start: 2 copper layers, 122 parts, among them J1 31-5431-2010_CID2.5.196, J2 31-5431-2010_CID2.5.196, J3 31-5431-2010_CID2.5.196, J4 1945193_12P_CID2.2.928, J5 31-5431-2010_CID2.5.196, J6 31-5431-2010_CID2.5.196, U1 L7812ABD2T-TR_CID8.52.934, U2 MC7912ACD2TR4G_CID8.52.429, U3 LP2981IM5-5.0-NOPB_CID8.52.176, U5 TL084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

Commit message: Filters and tang nano 9k
Parts:
- added C49: C_0805_100nF_16V_X7R_CID1.2.3078, dtuspace_ipc:C0805_CAPC200X125X130L45N, F.Cu at (192.6, 57.1)
- added C50: C_0805_100nF_16V_X7R_CID1.2.3078, dtuspace_ipc:C0805_CAPC200X125X130L45N, F.Cu at (192.6, 60.0)
- added C51: C_2917_47uF_20V_20%_CID1.3.892, dtuspace_ipc:C2917_CAPC730X430X310L130N, F.Cu at (158.3, 36.8)
- added C52: C_2917_47uF_20V_20%_CID1.3.892, dtuspace_ipc:C2917_CAPC730X430X310L130N, F.Cu at (158.3, 42.9)
- added C53: C_2917_47uF_20V_20%_CID1.3.892, dtuspace_ipc:C2917_CAPC730X430X310L130N, F.Cu at (158.3, 48.9)
- added C54: C_2917_47uF_20V_20%_CID1.3.892, dtuspace_ipc:C2917_CAPC730X430X310L130N, F.Cu at (158.3, 55.0)
- added L1: L_3.3uH_870mA_CID7.3.944, dtuspace_ipc:L0805_INDC200X125X140L50N, F.Cu at (184.2, 50.0)
- added L2: L_3.3uH_870mA_CID7.3.944, dtuspace_ipc:L0805_INDC200X125X140L50N, F.Cu at (184.2, 52.9)
- added L3: L_3.3uH_870mA_CID7.3.944, dtuspace_ipc:L0805_INDC200X125X140L50N, F.Cu at (184.2, 55.8)
- added L4: L_3.3uH_870mA_CID7.3.944, dtuspace_ipc:L0805_INDC200X125X140L50N, F.Cu at (184.2, 58.7)
- added LD_SML-P11VTT86R1: ~, dtuspace_ipc:SML_P11, F.Cu at (267.0, 28.7)
- added LD_SML-P11VTT86R2: ~, dtuspace_ipc:SML_P11, F.Cu at (267.0, 30.4)
- added LD_SML-P11VTT86R3: ~, dtuspace_ipc:SML_P11, F.Cu at (267.0, 32.2)
- added LD_SML-P11VTT86R4: ~, dtuspace_ipc:SML_P11, F.Cu at (267.0, 34.0)
- added R53: R_0805_220R_CID10.9.602, dtuspace_ipc:R0805_RESC200X125X50L35N, F.Cu at (188.4, 49.9)
- added R54: R_0805_220R_CID10.9.602, dtuspace_ipc:R0805_RESC200X125X50L35N, F.Cu at (188.4, 52.8)
- added R55: R_0805_2M49_CID10.9.5964, dtuspace_ipc:R0805_RESC200X125X50L35N, F.Cu at (188.4, 55.7)
- added R56: R_0805_10M0_CID10.9.5993, dtuspace_ipc:R0805_RESC200X125X50L35N, F.Cu at (188.4, 58.5)
- moved J4 207.3 mm to (23.5, 98.5), turned to -90 degrees
- moved J1 172.0 mm to (47.0, 80.9)
- moved R52 148.7 mm to (94.5, 141.8), turned to 180 degrees
- moved R51 135.5 mm to (94.5, 111.8), turned to 180 degrees
- moved C2 95.5 mm to (76.0, 20.0)
- moved THS1 94.9 mm to (103.5, 27.9)
- moved R12 94.2 mm to (63.0, 136.0), turned to -90 degrees
- moved THS2 92.0 mm to (104.0, 38.0)
- moved OPA2 91.5 mm to (67.8, 140.2), turned to 180 degrees
- moved C9 89.1 mm to (105.0, 18.0)
- moved C17 84.4 mm to (55.5, 151.0), turned to -90 degrees
- moved C4 79.5 mm to (55.5, 122.0), turned to -90 degrees
- moved R1 79.0 mm to (53.0, 92.5)
- moved C3 78.2 mm to (55.5, 112.6), turned to 90 degrees
- moved OPA1 77.6 mm to (67.8, 111.7), turned to 180 degrees
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Connections:
- C47 pad 2: Net-(U6-CH0) -> Net-(C47-Pad2)
- C48 pad 1: +15V -> Net-(U7-Vin)
- C5 pad 2: +15V -> Net-(U1-VIN)
- C6 pad 1: +15V -> Net-(U3-ON/OFF)
- C7 pad 1: -15V -> Net-(U2-VIN)
- J5 pad 1: Net-(U6-CH0) -> Net-(C47-Pad2)
- R47 pad 2: Net-(U6-CH0) -> Net-(C47-Pad2)
- R52 pad 1: Net-(R52-Pad1) -> V_wire
- U1 pad 1: +15V -> Net-(U1-VIN)
- U2 pad 1: GND -> Net-(U2-VIN)
- U2 pad 3: -15V -> GND
- U3 pad 1: +15V -> Net-(U3-ON/OFF)
- U3 pad 3: +15V -> Net-(U3-ON/OFF)
- U5 pad 8: Net-(U6-CH0) -> Net-(C47-Pad2)
- U6 pad 3: unconnected-(U6-CH1-Pad3) -> Net-(U6-CH1)
- U7 pad 2: +15V -> Net-(U7-Vin)
Routing:
- net +10V: track 0.00 -> 97.9 mm
- net -10V: track 0.00 -> 87.7 mm, vias 0 -> 6
- net Net-(C1-Pad2): track 0.00 -> 59.8 mm, vias 0 -> 2
- net Net-(OPA1--): track 0.00 -> 25.2 mm
- net Net-(OPA2-Vo): track 0.00 -> 22.3 mm
- net Net-(OPA1-Vo): track 0.00 -> 21.8 mm
- net Net-(OPA2--): track 0.00 -> 18.5 mm
- net Net-(OPA1-+): track 0.00 -> 13.9 mm, vias 0 -> 2
- net Net-(J1-Pad1): track 0.00 -> 8.57 mm
