File: hb_chip_test/hb_chip_test.kicad_sch (KiCad schematic)
At the start: 138 parts, among them J1 31-5431-2010_CID2.5.196, J2 31-5431-2010_CID2.5.196, J3 31-5431-2010_CID2.5.196, J4 1945193_12P_CID2.2.928, J5 31-5431-2010_CID2.5.196, J6 31-5431-2010_CID2.5.196, U1 L7812ABD2T-TR_CID8.52.934, U2 MC7912ACD2TR4G_CID8.52.429, U3 LP2981IM5-5.0-NOPB_CID8.52.176, U5 TL084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

Commit message: Filters and tang nano 9k
Parts:
- added R55: R_0805_2M49_CID10.9.5964, R0805_RESC200X125X50L35N, symbol 10-Resistor:R_0805_2M49_CID10.9.5964
- added R56: R_0805_10M0_CID10.9.5993, R0805_RESC200X125X50L35N, symbol 10-Resistor:R_0805_10M0_CID10.9.5993
- added U8: Tang_Nano_9K, 0my_project:DIP-48_TangNano9K, symbol 0my_project:Tang_Nano_9K
- C51, C52, C53, C54: footprint C2917_CAPC730X430X310XL130N -> dtuspace_ipc:C2917_CAPC730X430X310L130N
- LD_SML-P11VTT86R1, LD_SML-P11VTT86R2, LD_SML-P11VTT86R3, LD_SML-P11VTT86R4: footprint (none) -> dtuspace_ipc:SML_P11; MPN (none) -> SML-P11VTT86R
Connections:
- net -12V: now also LD_SML-P11VTT86R3.1; no longer LD_SML-P11VTT86R3.
- net GND: now also LD_SML-P11VTT86R1.1, LD_SML-P11VTT86R2.1, LD_SML-P11VTT86R4.1, U2.3 (GND), R55.2; no longer LD_SML-P11VTT86R1., LD_SML-P11VTT86R2., LD_SML-P11VTT86R4., U2.1 (GND)
- net V_wire: now also R56.1; no longer R54.2
- net at R21.1: now also LD_SML-P11VTT86R2.2; no longer LD_SML-P11VTT86R2.
- net at R25.1: now also LD_SML-P11VTT86R3.2; no longer LD_SML-P11VTT86R3.
- net at R50.1: now also LD_SML-P11VTT86R4.2; no longer LD_SML-P11VTT86R4.
- net at C54.2, C7.1, L4.2: now also U2.1 (VIN); no longer U2.3 (VIN)
- net at R19.1: now also LD_SML-P11VTT86R1.2; no longer LD_SML-P11VTT86R1.
- new net: R54.2, R55.1, R56.2
Other:
- note removed: "RC led (~220 ohm, C?)"
- note removed: "spændingsdeler rc led"
- moved on the sheet: C24, C25, C26, C48, C49, C50, C51, J5, J6, JP1, L1, R19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
